File: kicad/mushroom_rocket/mushroom_rocket.kicad_sch (KiCad schematic)
At the start: 0 parts

Commit message: redesign of rocket
Parts:
- added BT1: Battery_Cell, blinkyparts:BatteryHolder_Keystone_1060_1x2032_HandSoldering, symbol Device:Battery_Cell
- added D1, D2, D3, D4: LED, blinkyparts:5mm_SMD-Pad, symbol Device:LED
- added SW1: SW_DIP_x01, blinkyparts:Push_Button, symbol Switch:SW_DIP_x01
Connections:
- new net +3V0: BT1.1 (+), SW1.2
- new net GND: BT1.2 (-), D1.2 (A), D2.2 (A), D3.2 (A), D4.2 (A)
- new net VCC: D1.1 (K), D2.1 (K), D3.1 (K), D4.1 (K), SW1.1
